File: Month01_UsbToSerial/UsbToSerial_v_0_2b.kicad_pcb (KiCad board)
At the start: 2 copper layers, 34.9 x 20.3 mm, 14 parts, among them J1 USB_B_Micro, J2 Conn_01x07_Female, J3 Conn_01x07_Female, U1 FT232RL

Commit message: Minor modification to V0.2b
Routing:
- net GNDREF: track 161.5 -> 162.9 mm
Other:
- board size 34.9 x 20.3 mm -> 33.7 x 20.3 mm
Changed lines of the file:
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@@
   (gr_circle (center 102.235 73.025) (end 102.489 73.025) (layer F.SilkS) (width 0.15))
   (gr_circle (center 101.092 73.152) (end 101.346 73.406) (layer F.Fab) (width 0.15))
-  (gr_text V.0.2b (at 77.47 88.265) (layer F.SilkS)
+  (gr_text V.0.2b (at 79.375 89.535 90) (layer F.SilkS)
     (effects (font (size 1 1) (thickness 0.15)) (justify left))
   )
-  (gr_line (start 76.835 90.17) (end 76.835 69.85) (layer Edge.Cuts) (width 0.2))
-  (gr_line (start 111.76 90.17) (end 76.835 90.17) (layer Edge.Cuts) (width 0.2))
+  (gr_line (start 78.105 90.17) (end 78.105 69.85) (layer Edge.Cuts) (width 0.2))
+  (gr_line (start 111.76 90.17) (end 78.105 90.17) (layer Edge.Cuts) (width 0.2))
   (gr_line (start 111.76 69.85) (end 111.76 90.17) (layer Edge.Cuts) (width 0.2))
-  (gr_line (start 76.835 69.85) (end 111.76 69.85) (layer Edge.Cuts) (width 0.2))
+  (gr_line (start 78.105 69.85) (end 111.76 69.85) (layer Edge.Cuts) (width 0.2))
   (segment (start 82.275 78.71) (end 82.095 78.71) (width 0.25) (layer F.Cu) (net 1))
   (segment (start 84.785 76.2) (end 82.275 78.71) (width 0.25) (layer F.Cu) (net 1))
@@
   (segment (start 84.360001 72.764003) (end 84.360001 71.149999) (width 0.25) (layer F.Cu) (net 2))
   (segment (start 82.975019 70.314979) (end 85.195021 70.314979) (width 0.25) (layer F.Cu) (net 2))
-  (segment (start 78.16999 79.506402) (end 78.16999 75.120008) (width 0.25) (layer F.Cu) (net 2))
-  (segment (start 80.72001 82.056422) (end 78.16999 79.506402) (width 0.25) (layer F.Cu) (net 2))
-  (segment (start 78.16999 75.120008) (end 82.975019 70.314979) (width 0.25) (layer F.Cu) (net 2))
-  (segment (start 80.72001 85.570012) (end 80.72001 82.056422) (width 0.25) (layer F.Cu) (net 2))
+  (segment (start 98.662938 89.705019) (end 84.855017 89.705019) (width 0.25) (layer F.Cu) (net 2))
   (segment (start 84.855017 89.705019) (end 80.72001 85.570012) (width 0.25) (layer F.Cu) (net 2))
-  (segment (start 98.662938 89.705019) (end 84.855017 89.705019) (width 0.25) (layer F.Cu) (net 2))
+  (segment (start 80.72001 72.569988) (end 80.72001 78.49858) (width 0.25) (layer F.Cu) (net 2))
+  (segment (start 82.975019 70.314979) (end 80.72001 72.569988) (width 0.25) (layer F.Cu) (net 2))
+  (segment (start 80.72001 85.570012) (end 80.72001 78.49858) (width 0.25) (layer F.Cu) (net 2))
+  (segment (start 80.72001 78.49858) (end 80.72001 82.056422) (width 0.25) (layer F.Cu) (net 2))
   (segment (start 108.89 76.53) (end 108.89 75.565) (width 0.25) (layer F.Cu) (net 3))
   (segment (start 107.315 78.105) (end 108.89 76.53) (width 0.25) (layer F.Cu) (net 3))
